File: doorbellphat.brd (EAGLE design)
At the start: 30 x 65 mm, 11 parts, among them U1 LM2594MX-5.0/NOPBM08A_TEX-M

Commit message: first spin
Parts:
- added C3: 47uF, TBB - rcl:CAPPM7343X310N
- C1: device TBB - rcl:C1210K -> TBB - rcl:CAPPM7343X310N
- C2: device TBB - rcl:C1210K -> TBB - rcl:2312
- moved C1 4.00 mm to (11.0, 31.0), turned to 180 degrees
Connections:
- net +5V: now also C2.A; no longer C2.1
- net GND: now also C1.C, C2.C, C3.C; no longer C1.2, C2.2
- net N$5: now also C1.A, C3.A; no longer C1.1
Routing:
- net N$5: track 13.5 -> 21.2 mm
Changed lines of the file:
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@@
 <layer number="41" name="tRestrict" color="4" fill="10" visible="yes" active="yes"/>
 <layer number="42" name="bRestrict" color="1" fill="10" visible="yes" active="yes"/>
-<layer number="43" name="vRestrict" color="2" fill="10" visible="yes" active="yes"/>
+<layer number="43" name="vRestrict" color="2" fill="10" visible="no" active="yes"/>
 <layer number="44" name="Drills" color="7" fill="1" visible="no" active="yes"/>
-<layer number="45" name="Holes" color="7" fill="1" visible="yes" active="yes"/>
+<layer number="45" name="Holes" color="7" fill="1" visible="no" active="yes"/>
 <layer number="46" name="Milling" color="3" fill="1" visible="no" active="yes"/>
 <layer number="47" name="Measures" color="7" fill="1" visible="no" active="yes"/>
-<layer number="48" name="Document" color="7" fill="1" visible="yes" active="yes"/>
-<layer number="49" name="Reference" color="7" fill="1" visible="yes" active="yes"/>
+<layer number="48" name="Document" color="7" fill="1" visible="no" active="yes"/>
+<layer number="49" name="Reference" color="7" fill="1" visible="no" active="yes"/>
 <layer number="50" name="dxf" color="7" fill="1" visible="no" active="no"/>
-<layer number="51" name="tDocu" color="7" fill="1" visible="no" active="yes"/>
-<layer number="52" name="bDocu" color="7" fill="1" visible="no" active="yes"/>
+<layer number="51" name="tDocu" color="7" fill="1" visible="yes" active="yes"/>
+<layer number="52" name="bDocu" color="7" fill="1" visible="yes" active="yes"/>
 <layer number="56" name="wert" color="7" fill="1" visible="no" active="no"/>
 <layer number="88" name="SimResults" color="9" fill="1" visible="no" active="no"/>
@@
 <layer number="250" name="Descript" color="3" fill="1" visible="no" active="no"/>
 <layer number="251" name="SMDround" color="12" fill="11" visible="no" active="no"/>
-<layer number="254" name="OrgLBR" color="13" fill="1" visible="yes" active="yes"/>
+<layer number="254" name="OrgLBR" color="13" fill="1" visible="no" active="yes"/>
 </layers>
 <board>
@@
 <elements>
 <element name="J4" library="TBB - pinhead" library_urn="urn:adsk.eagle:library:19155912" package="2X20" package3d_urn="urn:adsk.eagle:package:19156100/1" value="" x="3.5" y="32.5" smashed="yes" rot="R90">
-<attribute name="NAME" x="8.325" y="32.1" size="1.27" layer="25" font="vector" ratio="13" rot="R90"/>
+<attribute name="NAME" x="7.825" y="24.6" size="1.27" layer="25" font="vector" ratio="13" rot="R90"/>
 <attribute name="VALUE" x="7.945" y="7.1" size="1.27" layer="27" rot="R90"/>
 </element>
@@
 <attribute name="NAME" x="9.0234" y="15.865" size="1.27" layer="25" font="vector" ratio="13" rot="SR0"/>
 </element>
-<element name="C1" library="TBB - rcl" package="C1210K" value="47uF" x="15" y="31" smashed="yes" rot="R90">
-<attribute name="DESCRIPTION" value="" x="15" y="31" size="1.778" layer="27" rot="R90" display="off"/>
-<attribute name="MANUFACTURER" value="" x="15" y="31" size="1.778" layer="27" rot="R90" display="off"/>
-<attribute name="MFR_PART_NO" value="" x="15" y="31" size="1.778" layer="27" rot="R90" display="off"/>
-<attribute name="NAME" x="12.95" y="30.1" size="1.27" layer="25" font="vector" ratio="13" rot="R90"/>
-<attribute name="PACKAGE" value="" x="15" y="31" size="1.778" layer="27" rot="R90" display="off"/>
-<attribute name="VALUE" x="17.575" y="29.4" size="1.016" layer="27" rot="R90"/>
-<attribute name="VENDOR" value="" x="15" y="31" size="1.778" layer="27" rot="R90" display="off"/>
-</element>
-<element name="C2" library="TBB - rcl" package="C1210K" value="6.8uF" x="15" y="18" smashed="yes" rot="R180">
-<attribute name="DESCRIPTION" value="" x="15" y="18" size="1.778" layer="27" rot="R180" display="off"/>
-<attribute name="MANUFACTURER" value="" x="15" y="18" size="1.778" layer="27" rot="R180" display="off"/>
-<attribute name="MFR_PART_NO" value="" x="15" y="18" size="1.778" layer="27" rot="R180" display="off"/>
+<element name="C1" library="TBB - rcl" package="CAPPM7343X310N" value="47uF" x="11" y="31" smashed="yes" rot="R180">
+<attribute name="NAME" x="11.1" y="28.05" size="1.27" layer="25" font="vector" ratio="13" rot="R180"/>
+</element>
+<element name="C2" library="TBB - rcl" package="2312" value="6.8uF" x="15" y="18" smashed="yes" rot="R180">
 <attribute name="NAME" x="19.6" y="18.35" size="1.016" layer="25" font="vector" ratio="13" rot="R180"/>
-<attribute name="PACKAGE" value="" x="15" y="18" size="1.778" layer="27" rot="R180" display="off"/>
 <attribute name="VALUE" x="16.6" y="20.575" size="1.016" layer="27" rot="R180"/>
-<attribute name="VENDOR" value="" x="15" y="18" size="1.778" layer="27" rot="R180" display="off"/>
 </element>
 <element name="D2" library="diode" library_urn="urn:adsk.eagle:library:210" package="SMA" package3d_urn="urn:adsk.eagle:package:43460/3" value="SK220ATR" x="25" y="11" smashed="yes">
 <attribute name="NAME" x="24.15" y="13.5" size="1.27" layer="25" font="vector" ratio="13"/>
 <attribute name="POPULARITY" value="9" x="25" y="11" size="2.54" layer="27" font="vector" ratio="13" display="off"/>
-<attribute name="VALUE" x="22.25" y="7.5" size="1.27" layer="27" ratio="10"/>
 </element>
 <element name="F1" library="TBB - fuse" package="0603" value="125mA" x="24" y="26" smashed="yes" rot="R180">
@@
 <attribute name="VENDOR" value="DIGIKEY" x="24" y="26" size="1.27" layer="27" font="vector" ratio="13" rot="R180" display="off"/>
 </element>
+<element name="C3" library="TBB - rcl" package="CAPPM7343X310N" value="47uF" x="11" y="37" smashed="yes" rot="R180">
+<attribute name="NAME" x="18" y="38.35" size="1.27" layer="25" font="vector" ratio="13" rot="R180"/>
+</element>
 </elements>
 <signals>
@@
 <contactref element="J4" pad="4"/>
 <contactref element="J4" pad="2"/>
-<contactref element="C2" pad="1"/>
+<contactref element="C2" pad="A"/>
 <contactref element="L1" pad="1"/>
 <contactref element="U1" pad="4"/>
@@
 <vertex x="31" y="-1"/>
 </polygon>
-<wire x1="16.5" y1="18" x2="16.905" y2="18.405" width="0.6096" layer="1"/>
+<wire x1="17.338" y1="18" x2="16.905" y2="18.405" width="0.6096" layer="1"/>
 <wire x1="16.905" y1="18.405" x2="16.905" y2="21.17425" width="0.6096" layer="1"/>
-<wire x1="16.5" y1="18" x2="16.5" y2="16.9958" width="0.6096" layer="1"/>
+<wire x1="17.338" y1="18" x2="16.5" y2="16.9958" width="0.6096" layer="1"/>
 <wire x1="16.5" y1="16.9958" x2="10.5042" y2="11" width="0.6096" layer="1"/>
 <wire x1="10.5042" y1="11" x2="10.5042" y2="8.5042" width="0.6096" layer="1"/>
@@
 <contactref element="J4" pad="30"/>
 <contactref element="D1" pad="4"/>
-<contactref element="C1" pad="2"/>
+<contactref element="C1" pad="C"/>
 <contactref element="U1" pad="6"/>
-<contactref element="C2" pad="2"/>
+<contactref element="C2" pad="C"/>
 <polygon width="0.3048" layer="1">
 <vertex x="-1" y="-1"/>
@@
 </polygon>
 <contactref element="D2" pad="A"/>
+<contactref element="C3" pad="C"/>
 </signal>
 <signal name="N$1">
@@
 <contactref element="D1" pad="2_2"/>
 <contactref element="D1" pad="2_1"/>
-<contactref element="C1" pad="1"/>
+<contactref element="C1" pad="A"/>
 <contactref element="U1" pad="7"/>
-<wire x1="15" y1="29.5" x2="18.5" y2="29.5" width="0.6096" layer="1"/>
 <via x="18.5" y="29.5" extent="1-16" drill="0.35"/>
 <wire x1="18.5" y1="29.5" x2="22.2" y2="29.5" width="0.6096" layer="16"/>
@@
 <wire x1="22.25" y1="31" x2="22.25" y2="29.5" width="0.6096" layer="1"/>
 <wire x1="22.25" y1="29.5" x2="22.2" y2="29.5" width="0.6096" layer="1"/>
-<wire x1="14.365" y1="26.82575" x2="14.365" y2="29.5" width="0.6096" layer="1"/>
-<wire x1="14.365" y1="29.5" x2="15" y2="29.5" width="0.6096" layer="1"/>
 <wire x1="22.2625" y1="32.34" x2="22.2625" y2="31.2125" width="0.6096" layer="1"/>
 <wire x1="22.2625" y1="31.2125" x2="22.15" y2="31.1" width="0.6096" layer="1"/>
+<contactref element="C3" pad="A"/>
+<wire x1="14.1" y1="37" x2="14.1" y2="31" width="0.6096" layer="1"/>
+<wire x1="18.5" y1="29.5" x2="14.3" y2="29.5" width="0.6096" layer="1"/>
+<wire x1="14.3" y1="29.5" x2="14.3" y2="26.9139125" width="0.6096" layer="1"/>
+<wire x1="14.3" y1="26.9139125" x2="14.365" y2="26.8489125" width="0.6096" layer="1"/>
+<wire x1="14.365" y1="26.8489125" x2="14.365" y2="26.82575" width="0.6096" layer="1"/>
+<wire x1="14.1" y1="31" x2="14.1" y2="29.7" width="0.6096" layer="1"/>
+<wire x1="14.1" y1="29.7" x2="14.3" y2="29.5" width="0.6096" layer="1"/>
 </signal>
 <signal name="N$3">
