File: doorbellphat.sch (EAGLE design)
At the start: 11 parts, among them U1 LM2594MX-5.0/NOPBM08A_TEX-M

Commit message: first spin
Parts:
- added C3: 47uF, TBB - rcl:CPOL-US2917
- C1: device TBB - rcl:C-USC1210K -> TBB - rcl:CPOL-US2917
- C2: device TBB - rcl:C-USC1210K -> TBB - rcl:CPOL-US2312
Connections:
- net +5V: now also C2.+; no longer C2.1
- net GND: now also C1.-, C2.-, C3.-; no longer C1.2, C2.2
- net N$5: now also C1.+, C3.+; no longer C1.1

Commit message: added pn to capacitors and polarity to rear silkscreen
Parts:
- C1, C3: MFR_PART_NO (none) -> TAJD476M035RNJV
- C2: MFR_PART_NO (none) -> 293D685X9035C2TE3
Changed lines of the file:
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@@
 <grid distance="0.1" unitdist="inch" unit="inch" style="lines" multiple="1" display="no" altdistance="0.01" altunitdist="inch" altunit="inch"/>
 <layers>
-<layer number="1" name="Top" color="4" fill="1" visible="yes" active="no"/>
-<layer number="2" name="Route2" color="16" fill="1" visible="yes" active="no"/>
-<layer number="3" name="Route3" color="17" fill="1" visible="yes" active="no"/>
-<layer number="4" name="Route4" color="18" fill="1" visible="yes" active="no"/>
-<layer number="5" name="Route5" color="19" fill="1" visible="yes" active="no"/>
-<layer number="6" name="Route6" color="25" fill="1" visible="yes" active="no"/>
-<layer number="7" name="Route7" color="26" fill="1" visible="yes" active="no"/>
-<layer number="8" name="Route8" color="27" fill="1" visible="yes" active="no"/>
-<layer number="9" name="Route9" color="28" fill="1" visible="yes" active="no"/>
-<layer number="10" name="Route10" color="29" fill="1" visible="yes" active="no"/>
-<layer number="11" name="Route11" color="30" fill="1" visible="yes" active="no"/>
-<layer number="12" name="Route12" color="20" fill="1" visible="yes" active="no"/>
-<layer number="13" name="Route13" color="21" fill="1" visible="yes" active="no"/>
-<layer number="14" name="Route14" color="22" fill="1" visible="yes" active="no"/>
-<layer number="15" name="Route15" color="23" fill="1" visible="yes" active="no"/>
-<layer number="16" name="Bottom" color="1" fill="1" visible="yes" active="no"/>
-<layer number="17" name="Pads" color="2" fill="1" visible="yes" active="no"/>
-<layer number="18" name="Vias" color="2" fill="1" visible="yes" active="no"/>
-<layer number="19" name="Unrouted" color="6" fill="1" visible="yes" active="no"/>
-<layer number="20" name="Dimension" color="24" fill="1" visible="yes" active="no"/>
-<layer number="21" name="tPlace" color="7" fill="1" visible="yes" active="no"/>
-<layer number="22" name="bPlace" color="7" fill="1" visible="yes" active="no"/>
-<layer number="23" name="tOrigins" color="15" fill="1" visible="yes" active="no"/>
-<layer number="24" name="bOrigins" color="15" fill="1" visible="yes" active="no"/>
-<layer number="25" name="tNames" color="7" fill="1" visible="yes" active="no"/>
-<layer number="26" name="bNames" color="7" fill="1" visible="yes" active="no"/>
-<layer number="27" name="tValues" color="7" fill="1" visible="yes" active="no"/>
-<layer number="28" name="bValues" color="7" fill="1" visible="yes" active="no"/>
+<layer number="1" name="Top" color="4" fill="1" visible="no" active="no"/>
+<layer number="2" name="Route2" color="16" fill="1" visible="no" active="no"/>
+<layer number="3" name="Route3" color="17" fill="1" visible="no" active="no"/>
+<layer number="4" name="Route4" color="18" fill="1" visible="no" active="no"/>
+<layer number="5" name="Route5" color="19" fill="1" visible="no" active="no"/>
+<layer number="6" name="Route6" color="25" fill="1" visible="no" active="no"/>
+<layer number="7" name="Route7" color="26" fill="1" visible="no" active="no"/>
+<layer number="8" name="Route8" color="27" fill="1" visible="no" active="no"/>
+<layer number="9" name="Route9" color="28" fill="1" visible="no" active="no"/>
+<layer number="10" name="Route10" color="29" fill="1" visible="no" active="no"/>
+<layer number="11" name="Route11" color="30" fill="1" visible="no" active="no"/>
+<layer number="12" name="Route12" color="20" fill="1" visible="no" active="no"/>
+<layer number="13" name="Route13" color="21" fill="1" visible="no" active="no"/>
+<layer number="14" name="Route14" color="22" fill="1" visible="no" active="no"/>
+<layer number="15" name="Route15" color="23" fill="1" visible="no" active="no"/>
+<layer number="16" name="Bottom" color="1" fill="1" visible="no" active="no"/>
+<layer number="17" name="Pads" color="2" fill="1" visible="no" active="no"/>
+<layer number="18" name="Vias" color="2" fill="1" visible="no" active="no"/>
+<layer number="19" name="Unrouted" color="6" fill="1" visible="no" active="no"/>
+<layer number="20" name="Dimension" color="24" fill="1" visible="no" active="no"/>
+<layer number="21" name="tPlace" color="7" fill="1" visible="no" active="no"/>
+<layer number="22" name="bPlace" color="7" fill="1" visible="no" active="no"/>
+<layer number="23" name="tOrigins" color="15" fill="1" visible="no" active="no"/>
+<layer number="24" name="bOrigins" color="15" fill="1" visible="no" active="no"/>
+<layer number="25" name="tNames" color="7" fill="1" visible="no" active="no"/>
+<layer number="26" name="bNames" color="7" fill="1" visible="no" active="no"/>
+<layer number="27" name="tValues" color="7" fill="1" visible="no" active="no"/>
+<layer number="28" name="bValues" color="7" fill="1" visible="no" active="no"/>
 <layer number="29" name="tStop" color="7" fill="3" visible="no" active="no"/>
 <layer number="30" name="bStop" color="7" fill="6" visible="no" active="no"/>
@@
 <layer number="35" name="tGlue" color="7" fill="4" visible="no" active="no"/>
 <layer number="36" name="bGlue" color="7" fill="5" visible="no" active="no"/>
-<layer number="37" name="tTest" color="7" fill="1" visible="yes" active="no"/>
-<layer number="38" name="bTest" color="7" fill="1" visible="yes" active="no"/>
+<layer number="37" name="tTest" color="7" fill="1" visible="no" active="no"/>
+<layer number="38" name="bTest" color="7" fill="1" visible="no" active="no"/>
 <layer number="39" name="tKeepout" color="4" fill="11" visible="no" active="no"/>
 <layer number="40" name="bKeepout" color="1" fill="11" visible="no" active="no"/>
@@
 <layer number="44" name="Drills" color="7" fill="1" visible="no" active="no"/>
 <layer number="45" name="Holes" color="7" fill="1" visible="no" active="no"/>
-<layer number="46" name="Milling" color="3" fill="1" visible="yes" active="no"/>
-<layer number="47" name="Measures" color="7" fill="1" visible="yes" active="no"/>
-<layer number="48" name="Document" color="7" fill="1" visible="yes" active="no"/>
-<layer number="49" name="Reference" color="7" fill="1" visible="yes" active="no"/>
-<layer number="50" name="dxf" color="7" fill="1" visible="yes" active="no"/>
-<layer number="51" name="tDocu" color="7" fill="1" visible="yes" active="no"/>
-<layer number="52" name="bDocu" color="7" fill="1" visible="yes" active="no"/>
-<layer number="56" name="wert" color="7" fill="1" visible="yes" active="no"/>
+<layer number="46" name="Milling" color="3" fill="1" visible="no" active="no"/>
+<layer number="47" name="Measures" color="7" fill="1" visible="no" active="no"/>
+<layer number="48" name="Document" color="7" fill="1" visible="no" active="no"/>
+<layer number="49" name="Reference" color="7" fill="1" visible="no" active="no"/>
+<layer number="50" name="dxf" color="7" fill="1" visible="no" active="no"/>
+<layer number="51" name="tDocu" color="7" fill="1" visible="no" active="no"/>
+<layer number="52" name="bDocu" color="7" fill="1" visible="no" active="no"/>
+<layer number="56" name="wert" color="7" fill="1" visible="no" active="no"/>
 <layer number="88" name="SimResults" color="9" fill="1" visible="yes" active="yes"/>
 <layer number="89" name="SimProbes" color="9" fill="1" visible="yes" active="yes"/>
@@
 <attribute name="MFR_PART_NO" value="SRU1038-331Y"/>
 </part>
-<part name="C1" library="TBB - rcl" deviceset="CPOL-US" device="2917" value="47uF"/>
+<part name="C1" library="TBB - rcl" deviceset="CPOL-US" device="2917" value="47uF">
+<attribute name="MFR_PART_NO" value="TAJD476M035RNJV"/>
+</part>
 <part name="V10" library="TBB - supply" deviceset="GND" device=""/>
 <part name="V11" library="TBB - supply" deviceset="GND" device=""/>
-<part name="C2" library="TBB - rcl" deviceset="CPOL-US" device="2312" value="6.8uF"/>
+<part name="C2" library="TBB - rcl" deviceset="CPOL-US" device="2312" value="6.8uF">
+<attribute name="MFR_PART_NO" value="293D685X9035C2TE3"/>
+</part>
 <part name="V12" library="TBB - supply" deviceset="GND" device=""/>
 <part name="V13" library="TBB - supply" deviceset="+5V" device=""/>
@@
 <part name="V14" library="TBB - supply" deviceset="GND" device=""/>
 <part name="F1" library="TBB - fuse" deviceset="PICO3" device="" value="125mA"/>
-<part name="C3" library="TBB - rcl" deviceset="CPOL-US" device="2917" value="47uF"/>
+<part name="C3" library="TBB - rcl" deviceset="CPOL-US" device="2917" value="47uF">
+<attribute name="MFR_PART_NO" value="TAJD476M035RNJV"/>
+</part>
 </parts>
 <sheets>
@@
 <attribute name="NAME" x="89.916" y="76.835" size="1.778" layer="95"/>
 <attribute name="VALUE" x="89.916" y="72.009" size="1.778" layer="96"/>
+<attribute name="MFR_PART_NO" x="88.9" y="76.2" size="1.778" layer="96" display="off"/>
 </instance>
 <instance part="V10" gate="GND" x="88.9" y="60.96" smashed="yes">
@@
 <attribute name="NAME" x="224.536" y="66.675" size="1.778" layer="95"/>
 <attribute name="VALUE" x="224.536" y="61.849" size="1.778" layer="96"/>
+<attribute name="MFR_PART_NO" x="223.52" y="66.04" size="1.778" layer="96" display="off"/>
 </instance>
 <instance part="V12" gate="GND" x="223.52" y="60.96" smashed="yes">
@@
 <attribute name="NAME" x="100.076" y="76.835" size="1.778" layer="95"/>
 <attribute name="VALUE" x="100.076" y="72.009" size="1.778" layer="96"/>
+<attribute name="MFR_PART_NO" x="99.06" y="76.2" size="1.778" layer="96" display="off"/>
 </instance>
 </instances>
